Commit message: Arreglos sistema. Falla SLAM

File: src/diablo_test/urdf/diablo.urdf (robot description, URDF)
Before this commit: robot diablo_mesh, 15 links, 14 joints
Links:
- added link lidar_link
Joints:
- added joint base_to_lidar: type fixed, parent base_link, child lidar_link, origin xyz=0.09 0.0 0.22 rpy=0.0 0.0 0.0

Commit message: Arreglo sistema de comunicaciones. Se lanza todo correctamente

File: src/diablo_test/urdf/diablo.urdf (robot description, URDF)
Before this commit: robot diablo_mesh, 16 links, 15 joints
Links:
- added link base_footprint
Joints:
- added joint base_footprint_to_base_link: type fixed, parent base_footprint, child base_link, origin xyz=0 0 0 rpy=0 0 3.14159
- joint base_to_lidar: origin xyz=0.09 0.0 0.22 rpy=0.0 0.0 0.0 -> xyz=0.09 0.0 0.22 rpy=0.0 0.0 3.14159

Commit message: Arreglo llegada a posicion. Sistema de navegacion completo

File: src/diablo_test/urdf/diablo.urdf (robot description, URDF)
Before this commit: robot diablo_mesh, 17 links, 16 joints
Joints:
- joint base_footprint_to_base_link: origin xyz=0 0 0 rpy=0 0 3.14159 -> xyz=0 0 0.13 rpy=0 0 3.14159
- joint base_to_lidar: origin xyz=0.09 0.0 0.22 rpy=0.0 0.0 3.14159 -> xyz=-0.09 0.0 0.22 rpy=0.0 0.0 0.0

Commit message: Calibracion parametros. Arreglo visualizacion RVizz

File: src/diablo_test/urdf/diablo.urdf (robot description, URDF)
Before this commit: robot diablo_mesh, 17 links, 16 joints
Joints:
- joint base_footprint_to_base_link: origin xyz=0 0 0.13 rpy=0 0 3.14159 -> xyz=0 0 0.13 rpy=0 0 0
- joint base_to_lidar: origin xyz=-0.09 0.0 0.22 rpy=0.0 0.0 0.0 -> xyz=0.09 0.0 0.22 rpy=0.0 0.0 3.14159
- joint left_j1: type continuous -> fixed
- joint left_j2: type continuous -> fixed
- joint left_j3: type continuous -> fixed
- joint left_j4: type continuous -> fixed
- joint left_j5: type continuous -> fixed
- joint little_wheel_left_j1: type continuous -> fixed
- joint little_wheel_left_j2: type continuous -> fixed
- joint little_wheel_right_j1: type continuous -> fixed
- joint little_wheel_right_j2: type continuous -> fixed
- joint right_j1: type continuous -> fixed
- joint right_j2: type continuous -> fixed
- joint right_j3: type continuous -> fixed
- joint right_j4: type continuous -> fixed
- joint right_j5: type continuous -> fixed

Commit message: Arreglo pitch y levantamiento y filtrado lidar

File: src/diablo_test/urdf/diablo.urdf (robot description, URDF)
Before this commit: robot diablo_mesh, 17 links, 16 joints
Links:
- removed link base_footprint
Joints:
- removed joint base_footprint_to_base_link

Commit message: Reordenamiento repo

File: src/diablo_test/urdf/diablo.urdf (robot description, URDF)
Before this commit: robot diablo_mesh, 15 links, 14 joints
Links:
- added link base_footprint
- added link lidar_link
Joints:
- added joint base_footprint_to_base_link: type fixed, parent base_footprint, child base_link, origin xyz=0 0 0.13 rpy=0 0 0
- added joint base_to_lidar: type fixed, parent base_link, child lidar_link, origin xyz=0.09 0.0 0.22 rpy=0.0 0.0 3.14159
- joint left_j1: type continuous -> fixed
- joint left_j2: type continuous -> fixed
- joint left_j3: type continuous -> fixed
- joint left_j4: type continuous -> fixed
- joint left_j5: type continuous -> fixed
- joint little_wheel_left_j1: type continuous -> fixed
- joint little_wheel_left_j2: type continuous -> fixed
- joint little_wheel_right_j1: type continuous -> fixed
- joint little_wheel_right_j2: type continuous -> fixed
- joint right_j1: type continuous -> fixed
- joint right_j2: type continuous -> fixed
- joint right_j3: type continuous -> fixed
- joint right_j4: type continuous -> fixed
- joint right_j5: type continuous -> fixed
